Commit message: customized robot environment

File: resources/robots/a1/Arcus_12dof.urdf (robot description, URDF)
Before this commit: robot Arcus, 28 links, 27 joints
Joints:
- joint left_hip_roll_joint: limit lower=-0.5236 upper=2.9671 effort=88 velocity=32 -> lower=-0.5236 upper=2.9671 effort=139 velocity=20
- joint right_hip_roll_joint: limit lower=-2.9671 upper=0.5236 effort=88 velocity=32 -> lower=-2.9671 upper=0.5236 effort=139 velocity=20
