Commit message: g1_23dof_fixed

File: resources/robots/g1_description/g1_23dof.urdf (robot description, URDF)
Before this commit: robot g1_23dof, 33 links, 32 joints
Links:
- removed link waist_support_link
- removed link waist_yaw_fixed_link
- added link world
- link torso_link: mass 8.562 -> 6.78; geometry collision mesh filename=meshes/torso_link_23dof_rev_1_0.STL; visual mesh filename=meshes/torso_link_23dof_rev_1_0.STL
Joints:
- removed joint waist_support_joint
- removed joint waist_yaw_fixed_joint
- added joint floating_base_joint: type floating, parent world, child pelvis
- joint d435_joint: origin xyz=0.0576235 0.01753 0.41987 rpy=0 0.8307767239493009 0 -> xyz=0.0576235 0.01753 0.42987 rpy=0 0.8307767239493009 0
- joint head_joint: origin xyz=0.0039635 0 -0.054 rpy=0 0 0 -> xyz=0.0039635 0 -0.044 rpy=0 0 0
- joint imu_in_torso_joint: origin xyz=-0.03959 -0.00224 0.13792 rpy=0 0 0 -> xyz=-0.03959 -0.00224 0.14792 rpy=0 0 0
- joint left_hip_roll_joint: limit lower=-0.5236 upper=2.9671 effort=88 velocity=32 -> lower=-0.5236 upper=2.9671 effort=139 velocity=20
- joint left_shoulder_pitch_joint: origin xyz=0.0039563 0.10022 0.23778 rpy=0.27931 5.4949E-05 -0.00019159 -> xyz=0.0039563 0.10022 0.24778 rpy=0.27931 5.4949E-05 -0.00019159
- joint logo_joint: origin xyz=0.0039635 0 -0.054 rpy=0 0 0 -> xyz=0.0039635 0 -0.044 rpy=0 0 0
- joint mid360_joint: origin xyz=0.0002835 0.00003 0.40618 rpy=0 0.04014257279586953 0 -> xyz=0.0002835 0.00003 0.41618 rpy=0 0.04014257279586953 0
- joint right_hip_roll_joint: limit lower=-2.9671 upper=0.5236 effort=88 velocity=32 -> lower=-2.9671 upper=0.5236 effort=139 velocity=20
- joint right_shoulder_pitch_joint: origin xyz=0.0039563 -0.10021 0.23778 rpy=-0.27931 5.4949E-05 0.00019159 -> xyz=0.0039563 -0.10021 0.24778 rpy=-0.27931 5.4949E-05 0.00019159
- joint waist_yaw_joint: origin xyz=-0.0039635 0 0.054 rpy=0 0 0 -> xyz=-0.0039635 0 0.044 rpy=0 0 0
